File: pcb/skibidi-album-clicker.kicad_sch (KiCad schematic)
At the start: 29 parts, among them J1 Conn_01x02_Socket, Q1 Q_PMOS_GSD, Q2 Q_NMOS_GSD, SW1 RotaryEncoder_Switch, U1 XIAO-RP2040-DIP, U2 MCP73831-2-OT

Commit message: add schematic
Other:
- company: (none) -> Toby Cm's Lab
- title: (none) -> skibidi-album-clicker
Changed lines of the file:
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@@
 	(generator_version "9.0")
 	(paper "A4")
+	(title_block
+		(title "skibidi-album-clicker")
+		(date "2025-12-14")
+		(rev "v3")
+		(company "Toby Cm's Lab")
+	)
 	(junction
 		(at 63.5 62.23)

Commit message: update
Parts:
- removed C2, C3: 4.7u, Capacitor_SMD:C_0603_1608Metric, symbol Device:C
- removed D1: LED, LED_SMD:LED_0603_1608Metric, symbol Device:LED
- removed D2: D_Schottky, Diode_SMD:D_SOD-123, symbol Device:D_Schottky
- removed H7, H8: MountingHole, MountingHole:MountingHole_2.2mm_M2_Pad, symbol Mechanical:MountingHole
- removed JP1: SolderJumper_2_Bridged, Jumper:SolderJumper-2_P1.3mm_Bridged_RoundedPad1.0x1.5mm, symbol Jumper:SolderJumper_2_Bridged
- removed JP2: SolderJumper_2_Open, Jumper:SolderJumper-2_P1.3mm_Open_RoundedPad1.0x1.5mm, symbol Jumper:SolderJumper_2_Open
- removed LED1: SK6812MINI-E, PCM_marbastlib-various:LED_6028R, symbol PCM_marbastlib-various:SK6812MINI-E
- removed Q1: Q_PMOS_GSD, Package_TO_SOT_SMD:SOT-23, symbol Transistor_FET:Q_PMOS_GSD
- removed Q2: Q_NMOS_GSD, Package_TO_SOT_SMD:SOT-23, symbol Transistor_FET:Q_NMOS_GSD
- removed U1: XIAO-RP2040-DIP, Seeed Studio XIAO Series Library:XIAO-RP2040-Simple-SMD, symbol Seeed_Studio_XIAO_Series:XIAO-RP2040-DIP
- removed U2: MCP73831-2-OT, Package_TO_SOT_SMD:SOT-23-5, symbol Battery_Management:MCP73831-2-OT
- added R6: 2.49k, Resistor_SMD:R_0603_1608Metric, symbol Device:R
- added SW2: K2-1102AQ-H4CW-01, easyeda2kicad:SW-TH_K2-1102BQ-G4CW-01, symbol easyeda2kicad:K2-1102AQ-H4CW-01
- added U1: PY25Q128HA-SUH-IR, Package_SO:SOIC-8_5.3x5.3mm_P1.27mm, symbol Memory_Flash:W25Q128JVS
- added U2: RP2040-ZERO, easyeda2kicad:COMM-SMD_RP2040-ZERO, symbol easyeda2kicad:RP2040-ZERO
- C1: value 4.7u -> 10u; LCSC Part (none) -> C96446
- C4: value 4.7u -> 100n; LCSC Part (none) -> C14663; now not fitted
- DS1: footprint misc:IPS LCD Display -> Connector_PinSocket_2.54mm:PinSocket_1x07_P2.54mm_Horizontal
- H3, H4: now not fitted
- H5: footprint MountingHole:MountingHole_2.2mm_M2_Pad -> MountingHole:MountingHole_3.2mm_M3_Pad; now not fitted
- H6: footprint MountingHole:MountingHole_2.2mm_M2_Pad -> MountingHole:MountingHole_3.2mm_M3_Pad
- R1, R2: value 2k -> 2.49k; footprint Resistor_SMD:R_0402_1005Metric -> Resistor_SMD:R_0603_1608Metric; LCSC Part (none) -> C2930072
- R3, R4, R5: value 100k -> 2.49k; footprint Resistor_SMD:R_0402_1005Metric -> Resistor_SMD:R_0603_1608Metric; LCSC Part (none) -> C2930072
- SW1: LCSC Part (none) -> C143801
Connections:
- net +BATT: now also R5.1
- net BLK: now also U2.15 (GP14)
- net DC: now also U2.14 (GP13)
- net GND: now also R4.2, SW1.S1, SW2.3, SW2.4, U1.4 (GND), U2.22 (GND); no longer C4.2, R1.2, R2.2, R5.2, SW1.S2
- net RES: now also U2.13 (GP12)
- net at R3.2: now also R4.1, SW2.1; no longer SW1.S1
- net +3V3: now reaches DS1.2 (VCC)
- net +3V3: now also C1.1, R1.1, R2.1, U1.8 (VCC), U2.21 (3V3)
- net SCK2: now reaches DS1.3 (SCL)
- net SCK2: now also U2.11 (GP10)
- net MOSI2: now reaches DS1.4 (SDA)
- net MOSI2: now also U2.12 (GP11)
- net A: now reaches SW1.A
- net A: now also U2.5 (GP4)
- net B: now reaches SW1.B
- net B: now also U2.6 (GP5)
- net +3.3V renamed B_VOLT
- net B_VOLT: now also R5.2, R6.1, U2.17 (GP26)
- removed net VBUS: C1.1, R4.1
- new net: R1.2, U1.3 (~{WP}/IO_{2})
- new net: R2.2, U1.7 (~{HOLD}/~{RESET}/IO_{3})
- new net +5V: U2.23 (5V)
- new net B_VOLT_REF: C4.2, R6.2, U2.16 (GP15)
- new net CS: U1.1 (~{CS}), U2.2 (GP1)
- new net E_SW: SW1.S2, U2.7 (GP6)
- new net LDO_CE: SW2.2, U2.20 (GP29)
- new net MISO: U1.2 (DO/IO_{1}), U2.1 (GP0)
- new net MOSI: U1.5 (DI/IO_{0}), U2.4 (GP3)
- new net SCK: U1.6 (CLK), U2.3 (GP2)
- no-connect marks 0 -> 5
Other:
- added sheet Charger (charger.kicad_sch)
- added sheet LDO (ldo.kicad_sch)
- moved on the sheet: J1

Commit message: finished routing yeahhhh
Signed-off-by: Toby Cm <toby@vsus.app>
Parts:
- removed SW1: RotaryEncoder_Switch, Rotary_Encoder:RotaryEncoder_Bourns_Vertical_PEC12R-3x17F-Sxxxx, symbol Device:RotaryEncoder_Switch
- added D2: SK6812MINI-E, LED_SMD:LED_SK6812MINI-E_3.2x2.8mm_P1.5mm_ReverseMount, symbol LED:SK6812MINI-E
- added SW1: RotaryEncoder_Switch_MP, Rotary_Encoder:RotaryEncoder_Bourns_Vertical_PEC12R-3x17F-Sxxxx, symbol Device:RotaryEncoder_Switch_MP
Connections:
- net A: now also SW1.A
- net B: now also SW1.B
- net E_SW: now also SW1.S2
- net GND: now also SW1.C, SW1.S1, SW1.SH
- net Neopixel: now reaches U2.8 (GP7)
- net Neopixel: now also D2.2 (DIN)
- no-connect marks 5 -> 4
